Commit message: feat(architecture): Initial SITL bringup, decoupled Redis state machine, and alpha-beta filter framework. See README for strict node boundaries.

File: src/drone_description/urdf/drone.urdf.xacro (robot description, xacro)
@@ -23,19 +23,4 @@
     <origin xyz="0 0 -0.05" rpy="0 0 0"/>
   </joint>
-  <link name="tether_dummy_link">
-    <inertial>
-      <mass value="0.01"/>
-      <origin xyz="0 0 0" rpy="0 0 0"/>
-      <inertia ixx="0.0001" ixy="0" ixz="0" iyy="0.0001" iyz="0" izz="0.0001"/>
-    </inertial>
-  </link>
-  <joint name="payload_swing_x" type="revolute">
-    <parent link="base_link"/>
-    <child link="tether_dummy_link"/>
-    <origin xyz="0 0 -0.08" rpy="0 0 0"/>
-    <axis xyz="1 0 0"/>
-    <limit lower="-0.25" upper="0.25" effort="10" velocity="5.0"/>
-    <dynamics damping="0.5" friction="0.1"/>
-  </joint>
   <link name="camera_link">
     <inertial>
@@ -48,11 +33,41 @@
     </visual>
   </link>
+  <joint name="camera_joint" type="fixed">
+    <parent link="base_link"/>
+    <child link="camera_link"/>
+    <origin xyz="0 0 -0.05" rpy="0 1.570796 0"/>
+  </joint>
+  <link name="tether_dummy_link">
+    <inertial>
+      <mass value="0.001"/>
+      <origin xyz="0 0 0" rpy="0 0 0"/>
+      <inertia ixx="0.00001" ixy="0" ixz="0" iyy="0.00001" iyz="0" izz="0.00001"/>
+    </inertial>
+  </link>
+  <joint name="payload_swing_x" type="revolute">
+    <parent link="base_link"/>
+    <child link="tether_dummy_link"/>
+    <origin xyz="0 0 -0.08" rpy="0 0 0"/>
+    <axis xyz="1 0 0"/>
+    <limit lower="-0.5" upper="0.5" effort="10" velocity="5.0"/>
+    <dynamics damping="0.1" friction="0.0"/>
+  </joint>
+  <link name="payload_link">
+    <inertial>
+      <mass value="1.0"/> <origin xyz="0 0 -0.25" rpy="0 0 0"/>
+      <inertia ixx="0.01" ixy="0" ixz="0" iyy="0.01" iyz="0" izz="0.01"/>
+    </inertial>
+    <visual>
+      <origin xyz="0 0 -0.25" rpy="0 0 0"/>
+      <geometry><box size="0.1 0.1 0.1"/></geometry>
+    </visual>
+  </link>
   <joint name="payload_swing_y" type="revolute">
     <parent link="tether_dummy_link"/>
-    <child link="camera_link"/>
-    <origin xyz="0 0 0" rpy="0 1.570796 0"/>
+    <child link="payload_link"/>
+    <origin xyz="0 0 0" rpy="0 0 0"/>
     <axis xyz="0 1 0"/>
-    <limit lower="-0.25" upper="0.25" effort="10" velocity="5.0"/>
-    <dynamics damping="0.5" friction="0.1"/>
+    <limit lower="-0.5" upper="0.5" effort="10" velocity="5.0"/>
+    <dynamics damping="0.1" friction="0.0"/>
   </joint>
   <xacro:macro name="rotor" params="motor_number x_pos y_pos">

Commit message: feat(architecture): key chnages to the antisway mechnais and maths and to the mavros

File: src/drone_description/urdf/drone.urdf.xacro (robot description, xacro)
@@ -55,5 +55,6 @@
   <link name="payload_link">
     <inertial>
-      <mass value="1.0"/> <origin xyz="0 0 -0.25" rpy="0 0 0"/>
+      <mass value="1.0"/>
+      <origin xyz="0 0 -0.25" rpy="0 0 0"/>
       <inertia ixx="0.01" ixy="0" ixz="0" iyy="0.01" iyz="0" izz="0.01"/>
     </inertial>
@@ -89,5 +90,9 @@
     </joint>
   </xacro:macro>
-  <xacro:rotor motor_number="0" x_pos="0.2" y_pos="-0.2"/>  <xacro:rotor motor_number="1" x_pos="-0.2" y_pos="0.2"/>  <xacro:rotor motor_number="2" x_pos="0.2" y_pos="0.2"/>   <xacro:rotor motor_number="3" x_pos="-0.2" y_pos="-0.2"/> <gazebo>
+  <xacro:rotor motor_number="0" x_pos="0.2" y_pos="-0.2"/>
+  <xacro:rotor motor_number="1" x_pos="-0.2" y_pos="0.2"/>
+  <xacro:rotor motor_number="2" x_pos="0.2" y_pos="0.2"/>
+  <xacro:rotor motor_number="3" x_pos="-0.2" y_pos="-0.2"/>
+  <gazebo>
     <plugin name="ardupilot_plugin" filename="libArduPilotPlugin.so">
       <fdm_addr>127.0.0.1</fdm_addr>
@@ -133,5 +138,6 @@
         <cmd_min>-2.5</cmd_min>
         <jointName>rotor_2_joint</jointName>
-        <multiplier>-838</multiplier> </control>
+        <multiplier>-838</multiplier>
+      </control>
       <control channel="3">
         <type>VELOCITY</type>
@@ -145,5 +151,6 @@
         <cmd_min>-2.5</cmd_min>
         <jointName>rotor_3_joint</jointName>
-        <multiplier>-838</multiplier> </control>
+        <multiplier>-838</multiplier>
+      </control>
     </plugin>
   </gazebo>

Commit message: Feat/drone bringup and infrastructure (#14)
* build: update docker environment for swarm simulation

* config: update base iris firmware parameters

* feat(drone_description): add URDF, launch files, and package configurations

* docs: update readme and repository metrics

* feat(architecture): Initial SITL bringup, decoupled Redis state machine, and alpha-beta filter framework. See README for strict node boundaries.

* feat(architecture): key chnages to the antisway mechnais and maths and to the mavros

---------

Co-authored-by: ASH-2012 <YOUR_GITHUB_EMAIL@example.com>

File: src/drone_description/urdf/drone.urdf.xacro (robot description, xacro)
@@ -23,19 +23,4 @@
     <origin xyz="0 0 -0.05" rpy="0 0 0"/>
   </joint>
-  <link name="tether_dummy_link">
-    <inertial>
-      <mass value="0.01"/>
-      <origin xyz="0 0 0" rpy="0 0 0"/>
-      <inertia ixx="0.0001" ixy="0" ixz="0" iyy="0.0001" iyz="0" izz="0.0001"/>
-    </inertial>
-  </link>
-  <joint name="payload_swing_x" type="revolute">
-    <parent link="base_link"/>
-    <child link="tether_dummy_link"/>
-    <origin xyz="0 0 -0.08" rpy="0 0 0"/>
-    <axis xyz="1 0 0"/>
-    <limit lower="-0.25" upper="0.25" effort="10" velocity="5.0"/>
-    <dynamics damping="0.5" friction="0.1"/>
-  </joint>
   <link name="camera_link">
     <inertial>
@@ -48,11 +33,42 @@
     </visual>
   </link>
+  <joint name="camera_joint" type="fixed">
+    <parent link="base_link"/>
+    <child link="camera_link"/>
+    <origin xyz="0 0 -0.05" rpy="0 1.570796 0"/>
+  </joint>
+  <link name="tether_dummy_link">
+    <inertial>
+      <mass value="0.001"/>
+      <origin xyz="0 0 0" rpy="0 0 0"/>
+      <inertia ixx="0.00001" ixy="0" ixz="0" iyy="0.00001" iyz="0" izz="0.00001"/>
+    </inertial>
+  </link>
+  <joint name="payload_swing_x" type="revolute">
+    <parent link="base_link"/>
+    <child link="tether_dummy_link"/>
+    <origin xyz="0 0 -0.08" rpy="0 0 0"/>
+    <axis xyz="1 0 0"/>
+    <limit lower="-0.5" upper="0.5" effort="10" velocity="5.0"/>
+    <dynamics damping="0.1" friction="0.0"/>
+  </joint>
+  <link name="payload_link">
+    <inertial>
+      <mass value="1.0"/>
+      <origin xyz="0 0 -0.25" rpy="0 0 0"/>
+      <inertia ixx="0.01" ixy="0" ixz="0" iyy="0.01" iyz="0" izz="0.01"/>
+    </inertial>
+    <visual>
+      <origin xyz="0 0 -0.25" rpy="0 0 0"/>
+      <geometry><box size="0.1 0.1 0.1"/></geometry>
+    </visual>
+  </link>
   <joint name="payload_swing_y" type="revolute">
     <parent link="tether_dummy_link"/>
-    <child link="camera_link"/>
-    <origin xyz="0 0 0" rpy="0 1.570796 0"/>
+    <child link="payload_link"/>
+    <origin xyz="0 0 0" rpy="0 0 0"/>
     <axis xyz="0 1 0"/>
-    <limit lower="-0.25" upper="0.25" effort="10" velocity="5.0"/>
-    <dynamics damping="0.5" friction="0.1"/>
+    <limit lower="-0.5" upper="0.5" effort="10" velocity="5.0"/>
+    <dynamics damping="0.1" friction="0.0"/>
   </joint>
   <xacro:macro name="rotor" params="motor_number x_pos y_pos">
@@ -74,5 +90,9 @@
     </joint>
   </xacro:macro>
-  <xacro:rotor motor_number="0" x_pos="0.2" y_pos="-0.2"/>  <xacro:rotor motor_number="1" x_pos="-0.2" y_pos="0.2"/>  <xacro:rotor motor_number="2" x_pos="0.2" y_pos="0.2"/>   <xacro:rotor motor_number="3" x_pos="-0.2" y_pos="-0.2"/> <gazebo>
+  <xacro:rotor motor_number="0" x_pos="0.2" y_pos="-0.2"/>
+  <xacro:rotor motor_number="1" x_pos="-0.2" y_pos="0.2"/>
+  <xacro:rotor motor_number="2" x_pos="0.2" y_pos="0.2"/>
+  <xacro:rotor motor_number="3" x_pos="-0.2" y_pos="-0.2"/>
+  <gazebo>
     <plugin name="ardupilot_plugin" filename="libArduPilotPlugin.so">
       <fdm_addr>127.0.0.1</fdm_addr>
@@ -118,5 +138,6 @@
         <cmd_min>-2.5</cmd_min>
         <jointName>rotor_2_joint</jointName>
-        <multiplier>-838</multiplier> </control>
+        <multiplier>-838</multiplier>
+      </control>
       <control channel="3">
         <type>VELOCITY</type>
@@ -130,5 +151,6 @@
         <cmd_min>-2.5</cmd_min>
         <jointName>rotor_3_joint</jointName>
-        <multiplier>-838</multiplier> </control>
+        <multiplier>-838</multiplier>
+      </control>
     </plugin>
   </gazebo>

Commit message: checkpoint: pre-T26 fix, R7 config validated

File: src/drone_description/urdf/drone.urdf.xacro (robot description, xacro)
@@ -27,6 +27,6 @@
     <sensor name="lidar_sensor" type="gpu_lidar">
       <always_on>true</always_on>
-      <visualize>true</visualize>
-      <update_rate>10</update_rate>
+      <visualize>false</visualize>
+      <update_rate>2</update_rate>
       <topic>lidar</topic>
       <lidar>
@@ -66,5 +66,5 @@
     <sensor name="camera_sensor" type="camera">
       <always_on>true</always_on>
-      <visualize>true</visualize>
+      <visualize>false</visualize>
       <update_rate>30</update_rate>
       <topic>camera/image</topic>
@@ -72,6 +72,6 @@
         <horizontal_fov>1.047</horizontal_fov>
         <image>
-          <width>640</width>
-          <height>480</height>
+          <width>320</width>
+          <height>240</height>
           <format>R8G8B8</format>
         </image>
@@ -139,6 +139,13 @@
   <xacro:rotor motor_number="2" x_pos="0.2" y_pos="0.2"/>
   <xacro:rotor motor_number="3" x_pos="-0.2" y_pos="-0.2"/>
+  <gazebo reference="base_link">
+    <sensor name="imu_sensor" type="imu">
+      <pose degrees="true">0 0 0 180 0 0</pose>
+      <always_on>1</always_on>
+      <update_rate>1000.0</update_rate>
+    </sensor>
+  </gazebo>
   <gazebo>
-    <plugin name="gz::sim::systems::ArduPilotSystem" filename="gz-sim-ardupilot-plugin">
+    <plugin name="ArduPilotPlugin" filename="ArduPilotPlugin">
       <fdm_addr>127.0.0.1</fdm_addr>
       <fdm_port_in>9002</fdm_port_in>
@@ -200,3 +207,43 @@
     </plugin>
   </gazebo>
+  <xacro:macro name="rotor_aero" params="motor_number chirality">
+    <plugin filename="gz-sim-lift-drag-system" name="gz::sim::systems::LiftDrag">
+      <a0>0.3</a0>
+      <alpha_stall>1.4</alpha_stall>
+      <cla>4.2500</cla>
+      <cda>0.10</cda>
+      <cma>0.0</cma>
+      <cla_stall>-0.025</cla_stall>
+      <cda_stall>0.0</cda_stall>
+      <cma_stall>0.0</cma_stall>
+      <area>0.00314</area>
+      <air_density>1.2041</air_density>
+      <cp>0.084 0 0</cp>
+      <forward>0 ${chirality} 0</forward>
+      <upward>0 0 1</upward>
+      <link_name>rotor_${motor_number}_link</link_name>
+    </plugin>
+    <plugin filename="gz-sim-lift-drag-system" name="gz::sim::systems::LiftDrag">
+      <a0>0.3</a0>
+      <alpha_stall>1.4</alpha_stall>
+      <cla>4.2500</cla>
+      <cda>0.10</cda>
+      <cma>0.0</cma>
+      <cla_stall>-0.025</cla_stall>
+      <cda_stall>0.0</cda_stall>
+      <cma_stall>0.0</cma_stall>
+      <area>0.00314</area>
+      <air_density>1.2041</air_density>
+      <cp>-0.084 0 0</cp>
+      <forward>0 ${-1 * chirality} 0</forward>
+      <upward>0 0 1</upward>
+      <link_name>rotor_${motor_number}_link</link_name>
+    </plugin>
+  </xacro:macro>
+  <gazebo>
+    <xacro:rotor_aero motor_number="0" chirality="1"/>
+    <xacro:rotor_aero motor_number="1" chirality="1"/>
+    <xacro:rotor_aero motor_number="2" chirality="-1"/>
+    <xacro:rotor_aero motor_number="3" chirality="-1"/>
+  </gazebo>
 </robot>

Commit message: T26: mitigate RTF/CPU cost of software rendering
- remove unused gpu_lidar sensor and its orphaned link/joint
- parametrize camera rate/resolution as xacro args (hw truth: 30Hz 320x240)
- sitl_bringup declares camera_rate launch arg, defaults 15 for GPU-less hosts
- export LP_NUM_THREADS=2 to stop llvmpipe saturating all 8 vCPUs
- flock single-instance guard keyed to DRONE_ID
- scoped Redis key clear on boot (fixes negative-age staleness across restarts)

Measured: gz CPU 199->130 pct, llvmpipe 124->56 pct, reproducible over 3 runs.
RTF mean varies 0.83-0.99 run-to-run on identical config; residual is host VM
scheduling, not addressable in-container.

File: src/drone_description/urdf/drone.urdf.xacro (robot description, xacro)
@@ -1,4 +1,7 @@
 <?xml version="1.0"?>
 <robot name="swarm_drone" xmlns:xacro="http://ros.org/wiki/xacro">
+  <xacro:arg name="camera_rate" default="30"/>
+  <xacro:arg name="camera_width" default="320"/>
+  <xacro:arg name="camera_height" default="240"/>
   <link name="base_link">
     <inertial>
@@ -17,34 +20,4 @@
     </collision>
   </link>
-  <link name="lidar_link"/>
-  <joint name="lidar_joint" type="fixed">
-    <parent link="base_link"/>
-    <child link="lidar_link"/>
-    <origin xyz="0 0 -0.05" rpy="0 0 0"/>
-  </joint>
-  <!-- Gazebo Harmonic Native Lidar Sensor -->
-  <gazebo reference="lidar_link">
-    <sensor name="lidar_sensor" type="gpu_lidar">
-      <always_on>true</always_on>
-      <visualize>false</visualize>
-      <update_rate>2</update_rate>
-      <topic>lidar</topic>
-      <lidar>
-        <scan>
-          <horizontal>
-            <samples>360</samples>
-            <resolution>1.0</resolution>
-            <min_angle>-3.14159</min_angle>
-            <max_angle>3.14159</max_angle>
-          </horizontal>
-        </scan>
-        <range>
-          <min>0.1</min>
-          <max>10.0</max>
-          <resolution>0.01</resolution>
-        </range>
-      </lidar>
-    </sensor>
-  </gazebo>
   <link name="camera_link">
     <inertial>
@@ -67,11 +40,11 @@
       <always_on>true</always_on>
       <visualize>false</visualize>
-      <update_rate>30</update_rate>
+      <update_rate>$(arg camera_rate)</update_rate>
       <topic>camera/image</topic>
       <camera>
         <horizontal_fov>1.047</horizontal_fov>
         <image>
-          <width>320</width>
-          <height>240</height>
+          <width>$(arg camera_width)</width>
+          <height>$(arg camera_height)</height>
           <format>R8G8B8</format>
         </image>

Commit message: fix(flight): close SITL actuation loop and resolve pre-arm/vision boot crashes
- urdf: strip zombie slung payload and joints to eliminate ground-plane physics chatter and gyro inconsistencies
- bringup: wire state_machine_node into swarm_bringup launch tree
- landing: gate touchdown cut-motors logic behind an explicit takeoff clearance threshold (z > 0.5m) to resolve B-00 boot latch
- state_machine: implement non-blocking service checks, 25s EKF boot settling, RC8 kill-threshold bump to 1900, and CommandTOL takeoff sequence
- vision: guard against OpenCV calcOpticalFlowPyrLK null pointers during ground near-clip and add feature re-seeding

File: src/drone_description/urdf/drone.urdf.xacro (robot description, xacro)
@@ -56,38 +56,4 @@
     </sensor>
   </gazebo>
-  <link name="tether_dummy_link">
-    <inertial>
-      <mass value="0.001"/>
-      <origin xyz="0 0 0" rpy="0 0 0"/>
-      <inertia ixx="0.00001" ixy="0" ixz="0" iyy="0.00001" iyz="0" izz="0.00001"/>
-    </inertial>
-  </link>
-  <joint name="payload_swing_x" type="revolute">
-    <parent link="base_link"/>
-    <child link="tether_dummy_link"/>
-    <origin xyz="0 0 -0.08" rpy="0 0 0"/>
-    <axis xyz="1 0 0"/>
-    <limit lower="-0.5" upper="0.5" effort="10" velocity="5.0"/>
-    <dynamics damping="0.1" friction="0.0"/>
-  </joint>
-  <link name="payload_link">
-    <inertial>
-      <mass value="1.0"/>
-      <origin xyz="0 0 -0.25" rpy="0 0 0"/>
-      <inertia ixx="0.01" ixy="0" ixz="0" iyy="0.01" iyz="0" izz="0.01"/>
-    </inertial>
-    <visual>
-      <origin xyz="0 0 -0.25" rpy="0 0 0"/>
-      <geometry><box size="0.1 0.1 0.1"/></geometry>
-    </visual>
-  </link>
-  <joint name="payload_swing_y" type="revolute">
-    <parent link="tether_dummy_link"/>
-    <child link="payload_link"/>
-    <origin xyz="0 0 0" rpy="0 0 0"/>
-    <axis xyz="0 1 0"/>
-    <limit lower="-0.5" upper="0.5" effort="10" velocity="5.0"/>
-    <dynamics damping="0.1" friction="0.0"/>
-  </joint>
   <xacro:macro name="rotor" params="motor_number x_pos y_pos">
     <link name="rotor_${motor_number}_link">

Commit message: feat(nav): establish decoupled GPS-denied VIO pipeline and single-writer control
- Decouple simulation transforms via gazebo_odom_adapter_node (NWU to ENU)
- Implement hardware-agnostic vio_bridge_node streaming 30Hz PoseStamped and TwistWithCovariance
- Configure ArduPilot EKF3 for pure external navigation (POSXY=6, VELXY=6, YAW=6, COMPASS_USE=0)
- Resolve topic contention in state_machine_node via /command/target_pose arbitration
- Fix vertical drift via 20Hz active position clamping in GUIDED mode
- Rewire altimeter_node to direct LaserScan rangefinder telemetry with NaN/inf filtering
- Recalibrate optical flow focal lengths (fx/fy=138.56) for 160x120 resolution in vision_nav_node
- Add timestamp age gating (<0.5s) and ground clamp (0.15m) to altitude-scaled flow
- Validate closed-loop kinematics: sub-millimeter hover and 3.71mm return error on 2x2m box trajectory

File: src/drone_description/urdf/drone.urdf.xacro (robot description, xacro)
@@ -87,4 +87,9 @@
   <gazebo>
     <plugin name="ArduPilotPlugin" filename="ArduPilotPlugin">
+      <sensor>
+        <type>rangefinder</type>
+        <index>1</index>
+        <topic>swarm_drone/rangefinder/scan</topic>
+      </sensor>
       <fdm_addr>127.0.0.1</fdm_addr>
       <fdm_port_in>9002</fdm_port_in>
@@ -186,3 +191,55 @@
     <xacro:rotor_aero motor_number="3" chirality="-1"/>
   </gazebo>
+  <!-- Downward Rangefinder Link and Sensor (Invariant I-1) -->
+  <link name="rangefinder_link">
+    <inertial>
+      <mass value="0.01"/>
+      <origin xyz="0 0 0" rpy="0 0 0"/>
+      <inertia ixx="0.00001" ixy="0" ixz="0" iyy="0.00001" iyz="0" izz="0.00001"/>
+    </inertial>
+  </link>
+  <joint name="rangefinder_joint" type="fixed">
+    <parent link="base_link"/>
+    <child link="rangefinder_link"/>
+    <origin xyz="0.05 0 -0.05" rpy="0 1.570796 0"/>
+  </joint>
+  <gazebo reference="rangefinder_link">
+    <sensor name="rangefinder_sensor" type="gpu_lidar">
+      <always_on>true</always_on>
+      <update_rate>30</update_rate>
+      <visualize>false</visualize>
+      <topic>swarm_drone/rangefinder/scan</topic>
+      <ray>
+        <scan>
+          <horizontal>
+            <samples>1</samples>
+            <resolution>1</resolution>
+            <min_angle>-0.01</min_angle>
+            <max_angle>0.01</max_angle>
+          </horizontal>
+          <vertical>
+            <samples>1</samples>
+            <resolution>1</resolution>
+            <min_angle>-0.01</min_angle>
+            <max_angle>0.01</max_angle>
+          </vertical>
+        </scan>
+        <range>
+          <min>0.01</min>
+          <max>40.0</max>
+          <resolution>0.01</resolution>
+        </range>
+      </ray>
+    </sensor>
+  </gazebo>
+  <gazebo>
+    <plugin
+      filename="gz-sim-odometry-publisher-system"
+      name="gz::sim::systems::OdometryPublisher">
+      <odom_topic>/model/swarm_drone/odometry</odom_topic>
+      <odom_frame>map</odom_frame>
+      <robot_base_frame>swarm_drone/base_link</robot_base_frame>
+      <dimensions>3</dimensions>
+    </plugin>
+  </gazebo>
 </robot>
