Commit message: Feat/gps denied vio navigation (#19)
* checkpoint: pre-T26 fix, R7 config validated

* T26: mitigate RTF/CPU cost of software rendering

- remove unused gpu_lidar sensor and its orphaned link/joint
- parametrize camera rate/resolution as xacro args (hw truth: 30Hz 320x240)
- sitl_bringup declares camera_rate launch arg, defaults 15 for GPU-less hosts
- export LP_NUM_THREADS=2 to stop llvmpipe saturating all 8 vCPUs
- flock single-instance guard keyed to DRONE_ID
- scoped Redis key clear on boot (fixes negative-age staleness across restarts)

Measured: gz CPU 199->130 pct, llvmpipe 124->56 pct, reproducible over 3 runs.
RTF mean varies 0.83-0.99 run-to-run on identical config; residual is host VM
scheduling, not addressable in-container.

* world: textured ground plane for optical flow (500 corners at 6m, was 0)

* fix(flight): close SITL actuation loop and resolve pre-arm/vision boot crashes

- urdf: strip zombie slung payload and joints to eliminate ground-plane physics chatter and gyro inconsistencies
- bringup: wire state_machine_node into swarm_bringup launch tree
- landing: gate touchdown cut-motors logic behind an explicit takeoff clearance threshold (z > 0.5m) to resolve B-00 boot latch
- state_machine: implement non-blocking service checks, 25s EKF boot settling, RC8 kill-threshold bump to 1900, and CommandTOL takeoff sequence
- vision: guard against OpenCV calcOpticalFlowPyrLK null pointers during ground near-clip and add feature re-seeding

* fix(perception): calibrate optical flow pipeline and align coordinate frames

- vision: replace ApproximateTimeSynchronizer with asynchronous ZOH sensor cache to restore 15Hz throughput
- vision: update focal length to analytic 277.13 and add dt factor to gyro de-rotation
- vision: remap camera optical axes to base_link body axes (-u -> Vx, v -> Vy)
- vision: tune corner extraction (qualityLevel=0.02, maxCorners=250) achieving >200 features
- mission: set default target altitude to 1.5m to stop initial-condition landing latch
- state_machine: wire emergency_override channel to cmd_vel setpoint dispatcher

* feat(nav): establish decoupled GPS-denied VIO pipeline and single-writer control

- Decouple simulation transforms via gazebo_odom_adapter_node (NWU to ENU)
- Implement hardware-agnostic vio_bridge_node streaming 30Hz PoseStamped and TwistWithCovariance
- Configure ArduPilot EKF3 for pure external navigation (POSXY=6, VELXY=6, YAW=6, COMPASS_USE=0)
- Resolve topic contention in state_machine_node via /command/target_pose arbitration
- Fix vertical drift via 20Hz active position clamping in GUIDED mode
- Rewire altimeter_node to direct LaserScan rangefinder telemetry with NaN/inf filtering
- Recalibrate optical flow focal lengths (fx/fy=138.56) for 160x120 resolution in vision_nav_node
- Add timestamp age gating (<0.5s) and ground clamp (0.15m) to altitude-scaled flow
- Validate closed-loop kinematics: sub-millimeter hover and 3.71mm return error on 2x2m box trajectory

---------

Co-authored-by: dev <dev@local>

File: src/drone_description/urdf/drone.urdf.xacro (robot description, xacro)
@@ -1,4 +1,7 @@
 <?xml version="1.0"?>
 <robot name="swarm_drone" xmlns:xacro="http://ros.org/wiki/xacro">
+  <xacro:arg name="camera_rate" default="30"/>
+  <xacro:arg name="camera_width" default="320"/>
+  <xacro:arg name="camera_height" default="240"/>
   <link name="base_link">
     <inertial>
@@ -17,34 +20,4 @@
     </collision>
   </link>
-  <link name="lidar_link"/>
-  <joint name="lidar_joint" type="fixed">
-    <parent link="base_link"/>
-    <child link="lidar_link"/>
-    <origin xyz="0 0 -0.05" rpy="0 0 0"/>
-  </joint>
-  <!-- Gazebo Harmonic Native Lidar Sensor -->
-  <gazebo reference="lidar_link">
-    <sensor name="lidar_sensor" type="gpu_lidar">
-      <always_on>true</always_on>
-      <visualize>true</visualize>
-      <update_rate>10</update_rate>
-      <topic>lidar</topic>
-      <lidar>
-        <scan>
-          <horizontal>
-            <samples>360</samples>
-            <resolution>1.0</resolution>
-            <min_angle>-3.14159</min_angle>
-            <max_angle>3.14159</max_angle>
-          </horizontal>
-        </scan>
-        <range>
-          <min>0.1</min>
-          <max>10.0</max>
-          <resolution>0.01</resolution>
-        </range>
-      </lidar>
-    </sensor>
-  </gazebo>
   <link name="camera_link">
     <inertial>
@@ -66,12 +39,12 @@
     <sensor name="camera_sensor" type="camera">
       <always_on>true</always_on>
-      <visualize>true</visualize>
-      <update_rate>30</update_rate>
+      <visualize>false</visualize>
+      <update_rate>$(arg camera_rate)</update_rate>
       <topic>camera/image</topic>
       <camera>
         <horizontal_fov>1.047</horizontal_fov>
         <image>
-          <width>640</width>
-          <height>480</height>
+          <width>$(arg camera_width)</width>
+          <height>$(arg camera_height)</height>
           <format>R8G8B8</format>
         </image>
@@ -83,38 +56,4 @@
     </sensor>
   </gazebo>
-  <link name="tether_dummy_link">
-    <inertial>
-      <mass value="0.001"/>
-      <origin xyz="0 0 0" rpy="0 0 0"/>
-      <inertia ixx="0.00001" ixy="0" ixz="0" iyy="0.00001" iyz="0" izz="0.00001"/>
-    </inertial>
-  </link>
-  <joint name="payload_swing_x" type="revolute">
-    <parent link="base_link"/>
-    <child link="tether_dummy_link"/>
-    <origin xyz="0 0 -0.08" rpy="0 0 0"/>
-    <axis xyz="1 0 0"/>
-    <limit lower="-0.5" upper="0.5" effort="10" velocity="5.0"/>
-    <dynamics damping="0.1" friction="0.0"/>
-  </joint>
-  <link name="payload_link">
-    <inertial>
-      <mass value="1.0"/>
-      <origin xyz="0 0 -0.25" rpy="0 0 0"/>
-      <inertia ixx="0.01" ixy="0" ixz="0" iyy="0.01" iyz="0" izz="0.01"/>
-    </inertial>
-    <visual>
-      <origin xyz="0 0 -0.25" rpy="0 0 0"/>
-      <geometry><box size="0.1 0.1 0.1"/></geometry>
-    </visual>
-  </link>
-  <joint name="payload_swing_y" type="revolute">
-    <parent link="tether_dummy_link"/>
-    <child link="payload_link"/>
-    <origin xyz="0 0 0" rpy="0 0 0"/>
-    <axis xyz="0 1 0"/>
-    <limit lower="-0.5" upper="0.5" effort="10" velocity="5.0"/>
-    <dynamics damping="0.1" friction="0.0"/>
-  </joint>
   <xacro:macro name="rotor" params="motor_number x_pos y_pos">
     <link name="rotor_${motor_number}_link">
@@ -139,6 +78,18 @@
   <xacro:rotor motor_number="2" x_pos="0.2" y_pos="0.2"/>
   <xacro:rotor motor_number="3" x_pos="-0.2" y_pos="-0.2"/>
+  <gazebo reference="base_link">
+    <sensor name="imu_sensor" type="imu">
+      <pose degrees="true">0 0 0 180 0 0</pose>
+      <always_on>1</always_on>
+      <update_rate>1000.0</update_rate>
+    </sensor>
+  </gazebo>
   <gazebo>
-    <plugin name="gz::sim::systems::ArduPilotSystem" filename="gz-sim-ardupilot-plugin">
+    <plugin name="ArduPilotPlugin" filename="ArduPilotPlugin">
+      <sensor>
+        <type>rangefinder</type>
+        <index>1</index>
+        <topic>swarm_drone/rangefinder/scan</topic>
+      </sensor>
       <fdm_addr>127.0.0.1</fdm_addr>
       <fdm_port_in>9002</fdm_port_in>
@@ -200,3 +151,95 @@
     </plugin>
   </gazebo>
+  <xacro:macro name="rotor_aero" params="motor_number chirality">
+    <plugin filename="gz-sim-lift-drag-system" name="gz::sim::systems::LiftDrag">
+      <a0>0.3</a0>
+      <alpha_stall>1.4</alpha_stall>
+      <cla>4.2500</cla>
+      <cda>0.10</cda>
+      <cma>0.0</cma>
+      <cla_stall>-0.025</cla_stall>
+      <cda_stall>0.0</cda_stall>
+      <cma_stall>0.0</cma_stall>
+      <area>0.00314</area>
+      <air_density>1.2041</air_density>
+      <cp>0.084 0 0</cp>
+      <forward>0 ${chirality} 0</forward>
+      <upward>0 0 1</upward>
+      <link_name>rotor_${motor_number}_link</link_name>
+    </plugin>
+    <plugin filename="gz-sim-lift-drag-system" name="gz::sim::systems::LiftDrag">
+      <a0>0.3</a0>
+      <alpha_stall>1.4</alpha_stall>
+      <cla>4.2500</cla>
+      <cda>0.10</cda>
+      <cma>0.0</cma>
+      <cla_stall>-0.025</cla_stall>
+      <cda_stall>0.0</cda_stall>
+      <cma_stall>0.0</cma_stall>
+      <area>0.00314</area>
+      <air_density>1.2041</air_density>
+      <cp>-0.084 0 0</cp>
+      <forward>0 ${-1 * chirality} 0</forward>
+      <upward>0 0 1</upward>
+      <link_name>rotor_${motor_number}_link</link_name>
+    </plugin>
+  </xacro:macro>
+  <gazebo>
+    <xacro:rotor_aero motor_number="0" chirality="1"/>
+    <xacro:rotor_aero motor_number="1" chirality="1"/>
+    <xacro:rotor_aero motor_number="2" chirality="-1"/>
+    <xacro:rotor_aero motor_number="3" chirality="-1"/>
+  </gazebo>
+  <!-- Downward Rangefinder Link and Sensor (Invariant I-1) -->
+  <link name="rangefinder_link">
+    <inertial>
+      <mass value="0.01"/>
+      <origin xyz="0 0 0" rpy="0 0 0"/>
+      <inertia ixx="0.00001" ixy="0" ixz="0" iyy="0.00001" iyz="0" izz="0.00001"/>
+    </inertial>
+  </link>
+  <joint name="rangefinder_joint" type="fixed">
+    <parent link="base_link"/>
+    <child link="rangefinder_link"/>
+    <origin xyz="0.05 0 -0.05" rpy="0 1.570796 0"/>
+  </joint>
+  <gazebo reference="rangefinder_link">
+    <sensor name="rangefinder_sensor" type="gpu_lidar">
+      <always_on>true</always_on>
+      <update_rate>30</update_rate>
+      <visualize>false</visualize>
+      <topic>swarm_drone/rangefinder/scan</topic>
+      <ray>
+        <scan>
+          <horizontal>
+            <samples>1</samples>
+            <resolution>1</resolution>
+            <min_angle>-0.01</min_angle>
+            <max_angle>0.01</max_angle>
+          </horizontal>
+          <vertical>
+            <samples>1</samples>
+            <resolution>1</resolution>
+            <min_angle>-0.01</min_angle>
+            <max_angle>0.01</max_angle>
+          </vertical>
+        </scan>
+        <range>
+          <min>0.01</min>
+          <max>40.0</max>
+          <resolution>0.01</resolution>
+        </range>
+      </ray>
+    </sensor>
+  </gazebo>
+  <gazebo>
+    <plugin
+      filename="gz-sim-odometry-publisher-system"
+      name="gz::sim::systems::OdometryPublisher">
+      <odom_topic>/model/swarm_drone/odometry</odom_topic>
+      <odom_frame>map</odom_frame>
+      <robot_base_frame>swarm_drone/base_link</robot_base_frame>
+      <dimensions>3</dimensions>
+    </plugin>
+  </gazebo>
 </robot>

Commit message: sim: landing legs give ToF 0.12 m ground clearance, victim decals flush at 2 mm; RNGFND1_GNDCLEAR 12; README section 17 arms on local position

File: src/drone_description/urdf/drone.urdf.xacro (robot description, xacro)
@@ -18,4 +18,20 @@
     <collision>
       <geometry><box size="0.4 0.4 0.1"/></geometry>
+    </collision>
+    <collision name="leg_fl">
+      <origin xyz="0.15 0.15 -0.11" rpy="0 0 0"/>
+      <geometry><box size="0.02 0.02 0.12"/></geometry>
+    </collision>
+    <collision name="leg_fr">
+      <origin xyz="0.15 -0.15 -0.11" rpy="0 0 0"/>
+      <geometry><box size="0.02 0.02 0.12"/></geometry>
+    </collision>
+    <collision name="leg_rl">
+      <origin xyz="-0.15 0.15 -0.11" rpy="0 0 0"/>
+      <geometry><box size="0.02 0.02 0.12"/></geometry>
+    </collision>
+    <collision name="leg_rr">
+      <origin xyz="-0.15 -0.15 -0.11" rpy="0 0 0"/>
+      <geometry><box size="0.02 0.02 0.12"/></geometry>
     </collision>
   </link>

Commit message: Phase 3: degraded estimation chain and hover gate (PASS) (#30)
* launch: onboard/sim split (I-8); use_sim_time and required integer drone_id

* sim: ros_imu -> /imu/raw with ICM-42688-P noise, base_link frame; camera 320x240@30 default; lidar max 4.0 m

* fcu: base_iris.param per README section 11 (GPS source removed, POSZ rangefinder); MAVROS deny-list removes GPS, second-source, ground-truth and second-actuator plugins

* sim: landing legs give ToF 0.12 m ground clearance, victim decals flush at 2 mm; RNGFND1_GNDCLEAR 12; README section 17 arms on local position

* sim: radar emulator (sigma 0.15 per Kramer, seeded bias_initial + bias walk, fault inflates R); gz --seed and SITL -w for reproducible runs

* estimation: robot_localization 15-state EKF per README section 6 (no absolute yaw, no accel, default Q) in swarm_bringup; vio_bridge relays /odometry/filtered to ExtNav

* guidance: pushpak_brain zero-velocity skeleton (sole cmd_vel writer, FS-5); arm_takeoff_handshake per section 17 with FS-4, opt-in via auto_takeoff; gate tolerance 0.8 m

* phase3: hover gate PASS (drift table, evaluator), backtrack_cov_threshold 0.2 with Q; T-2 fired, T-6 rig tripwire; LAND panic recorded

File: src/drone_description/urdf/drone.urdf.xacro (robot description, xacro)
@@ -18,4 +18,20 @@
     <collision>
       <geometry><box size="0.4 0.4 0.1"/></geometry>
+    </collision>
+    <collision name="leg_fl">
+      <origin xyz="0.15 0.15 -0.11" rpy="0 0 0"/>
+      <geometry><box size="0.02 0.02 0.12"/></geometry>
+    </collision>
+    <collision name="leg_fr">
+      <origin xyz="0.15 -0.15 -0.11" rpy="0 0 0"/>
+      <geometry><box size="0.02 0.02 0.12"/></geometry>
+    </collision>
+    <collision name="leg_rl">
+      <origin xyz="-0.15 0.15 -0.11" rpy="0 0 0"/>
+      <geometry><box size="0.02 0.02 0.12"/></geometry>
+    </collision>
+    <collision name="leg_rr">
+      <origin xyz="-0.15 -0.15 -0.11" rpy="0 0 0"/>
+      <geometry><box size="0.02 0.02 0.12"/></geometry>
     </collision>
   </link>
@@ -83,4 +99,24 @@
       <always_on>1</always_on>
       <update_rate>1000.0</update_rate>
+    </sensor>
+  </gazebo>
+  <gazebo reference="base_link">
+    <sensor name="ros_imu" type="imu">
+      <always_on>1</always_on>
+      <update_rate>200</update_rate>
+      <topic>swarm_drone/ros_imu</topic>
+      <gz_frame_id>base_link</gz_frame_id>
+      <imu>
+        <angular_velocity>
+          <x><noise type="gaussian"><mean>0.0</mean><stddev>6.91e-4</stddev></noise></x>
+          <y><noise type="gaussian"><mean>0.0</mean><stddev>6.91e-4</stddev></noise></y>
+          <z><noise type="gaussian"><mean>0.0</mean><stddev>6.91e-4</stddev></noise></z>
+        </angular_velocity>
+        <linear_acceleration>
+          <x><noise type="gaussian"><mean>0.0</mean><stddev>9.01e-3</stddev></noise></x>
+          <y><noise type="gaussian"><mean>0.0</mean><stddev>9.01e-3</stddev></noise></y>
+          <z><noise type="gaussian"><mean>0.0</mean><stddev>9.71e-3</stddev></noise></z>
+        </linear_acceleration>
+      </imu>
     </sensor>
   </gazebo>
@@ -227,5 +263,5 @@
         <range>
           <min>0.01</min>
-          <max>40.0</max>
+          <max>4.0</max>
           <resolution>0.01</resolution>
         </range>
